File: PCB/Projeto_Kicad/SCH-FLM-FTE12V-F3.kicad_sch (KiCad schematic)
At the start: 13 parts, among them J3 BPSC-2

Commit message: Atualização do resistor shunt R2 e R4
Parts:
- C7: value 100uF/25V -> 100uF/50V
Connections:
- net +15V renamed +18V
Changed lines of the file:
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@@
 			)
 		)
-		(property "Value" "+15V"
+		(property "Value" "+18V"
 			(at 124.46 133.096 0)
 			(show_name no)
@@
 			)
 		)
-		(property "Value" "100uF/25V"
+		(property "Value" "100uF/50V"
 			(at 136.398 159.004 90)
 			(show_name no)

Commit message: Atualização do arquivo 'FLM-FTE-SCH-01'
Other:
- note added: "STEP DOWN 18V - 12V"
- note removed: "STEP DOWN 15V - 12V"
Changed lines of the file:
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@@
 		)
 	)
-	(text "STEP DOWN 15V - 12V"
+	(text "STEP DOWN 18V - 12V"
 		(exclude_from_sim no)
 		(at 153.67 125.73 0)
