File: PCB/Projeto_Kicad/PCB-FLM-FTE-12V.kicad_pcb (KiCad board)
At the start: 2 copper layers, 120 x 75 mm, 54 parts, among them CN1 AKZ700-2-5,08V, CN2 AKZ700-2-5,08V, J1 BPSC-4, J2 MCS-6, J3 BPSC-2, Q1 TIP120, Q2 BC547, Q3 BC547, Q4 BC547, U1 ESP32-WROOM-32E-N8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

Commit message: Adição do R7 em paralelo com R6 e adição do RF2 de 15K e mudança de valor do RF1 de 10K para 15K
Parts:
- added R7: 0,22R/5W, Resistor_THT:R_Axial_DIN0516_L15.5mm_D5.0mm_P5.08mm_Vertical, F.Cu at (152.0, 62.9)
- C1, C5: value 4700uF/25V -> 4700uF/35V
- C7: value 100uF/25V -> 100uF/50V
- R2: value 0,44R/5W -> 0,33R/5W
- RV1: value 10K -> 11K
- moved C3 7.50 mm to (147.1, 38.3), turned to -90 degrees
- moved CN2 5.48 mm to (151.6, 57.4)
- moved R6 5.38 mm to (152.1, 68.7), turned to 180 degrees
- moved R2 4.89 mm to (151.5, 46.7)
Connections:
- net +15V renamed +18V
- R2 pad 2: Vout -> Net-(R2-Pad2)
- R6 pad 1: GND -> Ler_IRef
- R6 pad 2: Ler_IRef -> GND
Routing:
- net Net-(Q1-E): track 47.1 -> 40.6 mm
- net Ler_IRef: track 36.6 -> 42.3 mm
- added copper zone on F.Cu, net GND
Other:
- board text added: "R4"
- board text added: "RF2"
