File: PCB/Projeto_Kicad/PCB-FLM-FTE-12V.kicad_pcb (KiCad board)
At the start: 2 copper layers, 120 x 75 mm, 55 parts, among them CN1 AKZ700-2-5,08V, CN2 AKZ700-2-5,08V, J1 BPSC-4, J2 MCS-6, J3 BPSC-2, Q1 TIP120, Q2 BC547, Q3 BC547, Q4 BC547, U1 ESP32-WROOM-32E-N8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

Commit message: Remoção dos Jumpers no TopSilkscreen
Other:
- board text removed: "JP1"
- board text removed: "JP2"
- board text removed: "JP3"
- board text removed: "JP4"
Changed lines of the file:
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@@
 			(drillshape 0)
 			(scaleselection 1)
-			(outputdirectory "../.plotacao/SVG/")
+			(outputdirectory "//192.168.1.254/wirebus/Usuários/Felipe/")
 		)
 	)
@@
 		)
 	)
-	(gr_line
-		(start 97.145 91.515)
-		(end 97.135 103.165)
-		(stroke
-			(width 0.15)
-			(type default)
-		)
-		(layer "F.SilkS")
-	)
-	(gr_line
-		(start 99.915 103.075)
-		(end 99.915 91.675)
-		(stroke
-			(width 0.15)
-			(type default)
-		)
-		(layer "F.SilkS")
-	)
-	(gr_line
-		(start 111.125 72.925)
-		(end 155.865 72.955)
-		(stroke
-			(width 0.15)
-			(type default)
-		)
-		(layer "F.SilkS")
-	)
-	(gr_line
-		(start 155.135 101.455)
-		(end 155.135 91.045)
-		(stroke
-			(width 0.15)
-			(type default)
-		)
-		(layer "F.SilkS")
-	)
-	(gr_line
-		(start 158.195 91.225)
-		(end 158.195 101.455)
-		(stroke
-			(width 0.15)
-			(type default)
-		)
-		(layer "F.SilkS")
-	)
-	(gr_line
-		(start 161.145 82.175)
-		(end 161.155 101.535)
-		(stroke
-			(width 0.15)
-			(type default)
-		)
-		(layer "F.SilkS")
-	)
 	(gr_rect
 		(start 46.706666 33.585333)
@@
 		)
 	)
-	(gr_text "JP1"
-		(at 93.725 98.485 0)
-		(layer "F.SilkS")
-		(effects
-			(font
-				(size 1 1)
-				(thickness 0.15)
-			)
-			(justify left bottom)
-		)
-	)
-	(gr_text "JP2"
-		(at 100.745 98.485 0)
-		(layer "F.SilkS")
-		(effects
-			(font
-				(size 1 1)
-				(thickness 0.15)
-			)
-			(justify left bottom)
-		)
-	)
-	(gr_text "JP4"
-		(at 109.625 75.535 0)
-		(layer "F.SilkS")
-		(effects
-			(font
-				(size 1 1)
-				(thickness 0.15)
-			)
-			(justify left bottom)
-		)
-	)
 	(gr_text "3"
 		(at 137.325 52.435 0)
@@
 		)
 	)
-	(gr_text "JP2"
-		(at 153.535 104.015 0)
-		(layer "F.SilkS")
-		(effects
-			(font
-				(size 1 1)
-				(thickness 0.15)
-			)
-			(justify left bottom)
-		)
-	)
-	(gr_text "JP4"
-		(at 154.325 75.435 0)
-		(layer "F.SilkS")
-		(effects
-			(font
-				(size 1 1)
-				(thickness 0.15)
-			)
-			(justify left bottom)
-		)
-	)
-	(gr_text "JP1"
-		(at 156.685 104.015 0)
-		(layer "F.SilkS")
-		(effects
-			(font
-				(size 1 1)
-				(thickness 0.15)
-			)
-			(justify left bottom)
-		)
-	)
 	(gr_text "GND"
 		(at 157.125 80.275 0)
@@
 		(layer "F.SilkS")
 		(effects
-			(font
-				(size 1 1)
-				(thickness 0.15)
-			)
-			(justify left bottom)
-		)
-	)
-	(gr_text "JP3"
-		(at 161.745 92.655 0)
-		(layer "F.SilkS")
-		(effects
